File: pcb/BathroomFan/BathroomFan.kicad_pcb (KiCad board)
At the start: 2 copper layers, 76 x 106 mm, 16 parts, among them J1 Screw_Terminal_01x02, J2 Screw_Terminal_01x02, SW1 SW_SPST, U1 ESP32-DEVKIT-V1, U2 DHT11, U3 AC/DC Module 5V 700mA

Commit message: SCH and PCB: redistributed ESP32 pins for better layout, first version of layout finished
Parts:
- moved MS1 18.2 mm to (149.5, 108.0), turned to 180 degrees
Connections:
- U1 pad 11: /RGB_BLUE -> unconnected-(U1-D21-Pad11)
- U1 pad 26: unconnected-(U1-D14-Pad26) -> /RELAY
- U1 pad 28: unconnected-(U1-D13-Pad28) -> /MOTION_SENSOR
- U1 pad 3: unconnected-(U1-D15-Pad3) -> /RGB_RED
- U1 pad 4: /RGB_RED -> /RGB_GREEN
- U1 pad 5: /RELAY -> /RGB_BLUE
- U1 pad 8: /RGB_GREEN -> unconnected-(U1-D5-Pad8)
- U1 pad 9: /MOTION_SENSOR -> unconnected-(U1-D18-Pad9)
Routing:
- net /RELAY: track 0.00 -> 29.9 mm
- net /RGB_BLUE: track 0.00 -> 28.3 mm
- net /MOTION_SENSOR: track 0.00 -> 24.7 mm
- net GND: track 0.00 -> 24.4 mm, vias 0 -> 15
- net /RGB_GREEN: track 0.00 -> 20.1 mm
- net /DHT_DATA: track 0.00 -> 18.1 mm
- net /RGB_RED: track 0.00 -> 15.9 mm
- net +5V: track 79.7 -> 64.6 mm
- net +3V3: track 41.9 -> 43.1 mm
- added copper zone on B.Cu, net GND
- added copper zone on F.Cu, net GND
Other:
- board text added: "Bathroom Fan Controller V${REVISION} ${COMMENT1} ${COMPANY}"
- board text added: "D"
- board text added: "GND"
- board text added: "SIG"
- board text added: "VCC"
- board text added: "X"
